File: ESP-XBee.brd (EAGLE design)
At the start: 10 parts, among them SW1 434111043826

Commit message: final GERBER generated
Parts:
- added LOGO3: OSHW-LOGOS, SparkFun-Aesthetics:OSHW-LOGO-S
- renumbered U$1 to XBEE-BASE
Routing:
- net RESET: track 45.6 -> 47.1 mm, vias 3 -> 2
Other:
- board text added: "thingBotESP"
- board text added: "v0.1"
