File: ESP-XBee.sch (EAGLE design)
At the start: 10 parts, among them SW1 434111043826

Commit message: final GERBER generated
Parts:
- added LOGO3: OSHW-LOGOS, SparkFun-Aesthetics:OSHW-LOGOS
- renumbered U$1 to XBEE-BASE
