File: v1.1/thingBot-ESPv1P0.sch (KiCad schematic (older format))
At the start: 11 parts

Commit message: minor changes
Parts:
- gave numbers to parts that had none: 11
Connections:
- net CSO is gone; now on net CS0: U2.17 (CS0)
- net GND is gone; now on net GNDREF: C1.2, C2.2, R3.2, SW1.3 (C), SW2.2, U2.9 (GND)
- net GPI015 is gone; now on net GPIO13: U1.12 (CTS/DIO7)
- net ADC: now also U1.8 (RESERVED); no longer U1.11 (AD4/DIO4)
- net GPIO0: now also U1.17 (AD3/DIO3); no longer U1.18 (AD2/DIO2)
- net GPIO12: now also U1.15 (AD5/DIO5); no longer U1.16 (RTS/AD6/DIO6)
- net GPIO13: no longer U1.15 (AD5/DIO5)
- net GPIO15: now also U1.11 (AD4/DIO4)
- net GPIO16: now also U1.13 (ON/SLEEP); no longer U1.8 (RESERVED)
- net GPIO2: now also U1.18 (AD2/DIO2); no longer U1.17 (AD3/DIO3)
- net GPIO14: now reaches U2.5 (GPIO14)
- net GPIO14: now also U1.16 (RTS/AD6/DIO6)
- no-connect marks 0 -> 3
Changed lines of the file:
@@
 $EndDescr
 $Comp
-L Switch_SPDT_x2 SW?
+L Switch_SPDT_x2 SW1
 U 1 1 5899D87C
 P 4000 4050
-F 0 "SW?" H 3800 4200 50  0000 C CNN
+F 0 "SW1" H 3800 4200 50  0000 C CNN
 F 1 "Switch_SPDT_x2" H 3750 3900 50  0000 C CNN
 F 2 "" H 4000 4050 50  0000 C CNN
@@
 $EndComp
 $Comp
-L ESP-12E U?
+L ESP-12E U2
 U 1 1 589AC8FD
 P 7100 2300
-F 0 "U?" H 7100 2200 50  0000 C CNN
+F 0 "U2" H 7100 2200 50  0000 C CNN
 F 1 "ESP-12E" H 7100 2400 50  0000 C CNN
 F 2 "" H 7000 2100 50  0001 C CNN
@@
 VCC
 Text Label 6850 3450 1    60   ~ 0
-CSO
+CS0
 Text Label 6950 3450 1    60   ~ 0
 MISO
@@
 MISO
 $Comp
-L GNDREF #PWR?
+L GNDREF #PWR01
 U 1 1 589B06E0
 P 3100 3100
-F 0 "#PWR?" H 3100 3150 30  0001 C CNN
+F 0 "#PWR01" H 3100 3150 30  0001 C CNN
 F 1 "GNDREF" H 3100 2950 30  0001 C CNN
 F 2 "" H 3100 3100 60  0000 C CNN
@@
 Text Label 5250 2100 2    60   ~ 0
 GPIO4
+Text Label 5250 2300 2    60   ~ 0
+GPIO0
 Text Label 5250 2200 2    60   ~ 0
-GPIO0
-Text Label 5250 2300 2    60   ~ 0
 GPIO2
-Text Label 5250 2900 2    60   ~ 0
+Text Label 3100 2700 0    60   ~ 0
 ADC
 Text Label 5250 2400 2    60   ~ 0
+GPIO14
+Text Label 5250 2500 2    60   ~ 0
 GPIO12
-Text Label 5250 2500 2    60   ~ 0
-GPIO13
-Text Label 5250 2800 2    60   ~ 0
-GPI015
-$Comp
-L R R?
+Text Label 5250 2900 2    60   ~ 0
+GPIO15
+$Comp
+L R R4
 U 1 1 589B0B5C
 P 6500 4150
-F 0 "R?" V 6580 4150 50  0000 C CNN
+F 0 "R4" V 6580 4150 50  0000 C CNN
 F 1 "12K" V 6500 4150 50  0000 C CNN
 F 2 "" V 6430 4150 50  0000 C CNN
@@
 $EndComp
 $Comp
-L R R?
+L R R5
 U 1 1 589B0BBD
 P 6850 4200
-F 0 "R?" V 6930 4200 50  0000 C CNN
+F 0 "R5" V 6930 4200 50  0000 C CNN
 F 1 "12K" V 6850 4200 50  0000 C CNN
 F 2 "" V 6780 4200 50  0000 C CNN
@@
 RESET
 $Comp
-L SW_PUSH SW?
+L SW_PUSH SW2
 U 1 1 589B0EA5
 P 7300 4450
-F 0 "SW?" H 7450 4560 50  0000 C CNN
+F 0 "SW2" H 7450 4560 50  0000 C CNN
 F 1 "SW_PUSH" H 7300 4370 50  0000 C CNN
 F 2 "" H 7300 4450 50  0000 C CNN
@@
 $EndComp
 $Comp
-L CP1 C?
+L CP1 C1
 U 1 1 589B154F
 P 5750 4100
-F 0 "C?" H 5775 4200 50  0000 L CNN
+F 0 "C1" H 5775 4200 50  0000 L CNN
 F 1 "100uF" H 5775 4000 50  0000 L CNN
 F 2 "" H 5750 4100 50  0000 C CNN
@@
 GND
 $Comp
-L C C?
+L C C2
 U 1 1 589B1646
 P 6150 4150
-F 0 "C?" H 6175 4250 50  0000 L CNN
+F 0 "C2" H 6175 4250 50  0000 L CNN
 F 1 "1uF" H 6175 4050 50  0000 L CNN
 F 2 "" H 6188 4000 50  0000 C CNN
@@
 GND
 $Comp
-L R R?
+L R R3
 U 1 1 589B1A91
 P 5350 4150
-F 0 "R?" V 5430 4150 50  0000 C CNN
+F 0 "R3" V 5430 4150 50  0000 C CNN
 F 1 "12K" V 5350 4150 50  0000 C CNN
 F 2 "" V 5280 4150 50  0000 C CNN
@@
 GPIO15
 $Comp
-L R R?
+L R R2
 U 1 1 589B1D4C
 P 5050 4100
-F 0 "R?" V 5130 4100 50  0000 C CNN
+F 0 "R2" V 5130 4100 50  0000 C CNN
 F 1 "12K" V 5050 4100 50  0000 C CNN
 F 2 "" V 4980 4100 50  0000 C CNN
@@
 Text Label 4650 4400 1    60   ~ 0
 GND
-Text Label 3100 2700 0    60   ~ 0
+Text Label 5250 2700 2    60   ~ 0
 GPIO16
 Text Label 7600 4650 1    60   ~ 0
 GND
 $Comp
-L R R?
+L R R1
 U 1 1 589B4DA5
 P 4500 3950
-F 0 "R?" V 4580 3950 50  0000 C CNN
+F 0 "R1" V 4580 3950 50  0000 C CNN
 F 1 "12K" V 4500 3950 50  0000 C CNN
 F 2 "" V 4430 3950 50  0000 C CNN
@@
 VCC
 $Comp
-L XBEE_MODULE U?
+L XBEE_MODULE U1
 U 1 1 5899D937
 P 4150 2550
-F 0 "U?" H 4200 2500 60  0000 C CNN
+F 0 "U1" H 4200 2500 60  0000 C CNN
 F 1 "XBEE_MODULE" H 3750 3250 60  0000 C CNN
 F 2 "" H 4150 2550 60  0001 C CNN
@@
 	1    0    0    -1
 $EndComp
+Wire Wire Line
+	6200 2400 5950 2400
+Text Label 5950 2400 0    60   ~ 0
+GPIO14
+Text Label 5250 2800 2    60   ~ 0
+GPIO13
+Wire Wire Line
+	4950 2700 5250 2700
+Text Label 3100 2900 0    60   ~ 0
+GND
+NoConn ~ 7050 3200
+NoConn ~ 7150 3200
+NoConn ~ 4950 2600
 $EndSCHEMATC

Commit message: schematic verified
Parts:
- added D1: POWER_LED, LEDs:LED_0805, symbol LED
- added R6: 1K, Resistors_SMD:R_0805_HandSoldering, symbol R
- C1: footprint (none) -> Capacitors_SMD:C_1206_HandSoldering
- C2: footprint (none) -> Capacitors_SMD:C_0805_HandSoldering
- R1, R2, R3, R4, R5: footprint (none) -> Resistors_SMD:R_0805_HandSoldering
- SW1: footprint (none) -> Buttons_Switches_SMD:SW_SPDT_PCM12
- SW2: footprint (none) -> switches:SW_SPST_B3U-1000P_SUNROM
- U1: footprint (none) -> Xbee:XBee_Plug_without_Jtag
- U2: footprint (none) -> ESP8266:ESP-12E
Connections:
- net CH_PD: now also R4.2; no longer R4.1
- net GNDREF: now also D1.1 (K)
- net VCC renamed +3V3
- net +3V3: now also R4.1, R6.1; no longer R4.2
- new net: D1.2 (A), R6.2
Changed lines of the file:
@@
 F 0 "SW1" H 3800 4200 50  0000 C CNN
 F 1 "Switch_SPDT_x2" H 3750 3900 50  0000 C CNN
-F 2 "" H 4000 4050 50  0000 C CNN
+F 2 "Buttons_Switches_SMD:SW_SPDT_PCM12" H 4000 4050 50  0001 C CNN
 F 3 "" H 4000 4050 50  0000 C CNN
 	1    4000 4050
@@
 F 0 "U2" H 7100 2200 50  0000 C CNN
 F 1 "ESP-12E" H 7100 2400 50  0000 C CNN
-F 2 "" H 7000 2100 50  0001 C CNN
+F 2 "ESP8266:ESP-12E" H 7000 2100 50  0001 C CNN
 F 3 "" H 7100 2200 50  0001 C CNN
 F 4 "Ai-thinker" H 7200 2300 61  0001 C CNN "MFG_NAME"
@@
 Text Label 8250 2600 2    60   ~ 0
 GPIO15
-Text Label 8250 2700 2    60   ~ 0
-GND
 Text Label 5950 2000 0    60   ~ 0
 RESET
@@
 Text Label 5950 2600 0    60   ~ 0
 GPIO13
-Text Label 5950 2700 0    60   ~ 0
-VCC
 Text Label 6850 3450 1    60   ~ 0
 CS0
@@
 Text Label 7350 3450 1    60   ~ 0
 SCLK
-Text Label 3100 2000 0    60   ~ 0
-VCC
 Text Label 3100 2100 0    60   ~ 0
 TXD
@@
 F 0 "R4" V 6580 4150 50  0000 C CNN
 F 1 "12K" V 6500 4150 50  0000 C CNN
-F 2 "" V 6430 4150 50  0000 C CNN
+F 2 "Resistors_SMD:R_0805_HandSoldering" V 6430 4150 50  0001 C CNN
 F 3 "" H 6500 4150 50  0000 C CNN
 	1    6500 4150
@@
 F 0 "R5" V 6930 4200 50  0000 C CNN
 F 1 "12K" V 6850 4200 50  0000 C CNN
-F 2 "" V 6780 4200 50  0000 C CNN
+F 2 "Resistors_SMD:R_0805_HandSoldering" V 6780 4200 50  0001 C CNN
 F 3 "" H 6850 4200 50  0000 C CNN
 	1    6850 4200
 	1    0    0    -1
 $EndComp
-Text Label 6500 4500 1    60   ~ 0
-VCC
-Text Label 6500 3750 3    60   ~ 0
+Text Label 6500 4575 1    60   ~ 0
 CH_PD
 Text Label 6850 3750 3    60   ~ 0
@@
 F 0 "SW2" H 7450 4560 50  0000 C CNN
 F 1 "SW_PUSH" H 7300 4370 50  0000 C CNN
-F 2 "" H 7300 4450 50  0000 C CNN
+F 2 "switches:SW_SPST_B3U-1000P_SUNROM" H 7300 4450 50  0001 C CNN
 F 3 "" H 7300 4450 50  0000 C CNN
 	1    7300 4450
@@
 F 0 "C1" H 5775 4200 50  0000 L CNN
 F 1 "100uF" H 5775 4000 50  0000 L CNN
-F 2 "" H 5750 4100 50  0000 C CNN
+F 2 "Capacitors_SMD:C_1206_HandSoldering" H 5750 4100 50  0001 C CNN
 F 3 "" H 5750 4100 50  0000 C CNN
 	1    5750 4100
 	1    0    0    -1
 $EndComp
-Text Label 5750 3750 3    60   ~ 0
-VCC
-Text Label 5750 4500 1    60   ~ 0
-GND
 $Comp
 L C C2
@@
 F 0 "C2" H 6175 4250 50  0000 L CNN
 F 1 "1uF" H 6175 4050 50  0000 L CNN
-F 2 "" H 6188 4000 50  0000 C CNN
+F 2 "Capacitors_SMD:C_0805_HandSoldering" H 6188 4000 50  0001 C CNN
 F 3 "" H 6150 4150 50  0000 C CNN
 	1    6150 4150
@@
 Text Label 6150 3750 3    60   ~ 0
 RESET
-Text Label 6150 4500 1    60   ~ 0
-GND
 $Comp
 L R R3
@@
 F 0 "R3" V 5430 4150 50  0000 C CNN
 F 1 "12K" V 5350 4150 50  0000 C CNN
-F 2 "" V 5280 4150 50  0000 C CNN
+F 2 "Resistors_SMD:R_0805_HandSoldering" V 5280 4150 50  0001 C CNN
 F 3 "" H 5350 4150 50  0000 C CNN
 	1    5350 4150
 	1    0    0    -1
 $EndComp
-Text Label 5350 4500 1    60   ~ 0
-GND
 Text Label 5350 3700 3    60   ~ 0
 GPIO15
@@
 F 0 "R2" V 5130 4100 50  0000 C CNN
 F 1 "12K" V 5050 4100 50  0000 C CNN
-F 2 "" V 4980 4100 50  0000 C CNN
+F 2 "Resistors_SMD:R_0805_HandSoldering" V 4980 4100 50  0001 C CNN
 F 3 "" H 5050 4100 50  0000 C CNN
 	1    5050 4100
@@
 Text Label 5050 4500 1    60   ~ 0
 GPIO2
-Text Label 5050 3750 3    60   ~ 0
-VCC
 Text Label 3300 4050 0    60   ~ 0
 GPIO0
-Text Label 4650 4400 1    60   ~ 0
-GND
 Text Label 5250 2700 2    60   ~ 0
 GPIO16
-Text Label 7600 4650 1    60   ~ 0
-GND
 $Comp
 L R R1
@@
 F 0 "R1" V 4580 3950 50  0000 C CNN
 F 1 "12K" V 4500 3950 50  0000 C CNN
-F 2 "" V 4430 3950 50  0000 C CNN
+F 2 "Resistors_SMD:R_0805_HandSoldering" V 4430 3950 50  0001 C CNN
 F 3 "" H 4500 3950 50  0000 C CNN
 	1    4500 3950
@@
 	6200 2600 5950 2600
 Wire Wire Line
-	6200 2700 5950 2700
+	5800 2700 6200 2700
 Wire Wire Line
 	6850 3200 6850 3450
@@
 	6500 3750 6500 4000
 Wire Wire Line
-	6500 4300 6500 4500
+	6500 4300 6500 4575
 Wire Wire Line
 	6850 4050 6850 3750
@@
 	3700 4050 3300 4050
 Wire Wire Line
-	4300 4150 4650 4150
-Wire Wire Line
-	4650 4150 4650 4400
+	4300 4150 4700 4150
 Wire Wire Line
 	4300 3950 4350 3950
@@
 Wire Wire Line
 	4700 3950 4700 3750
-Text Label 4700 3750 3    60   ~ 0
-VCC
 $Comp
 L XBEE_MODULE U1
@@
 F 0 "U1" H 4200 2500 60  0000 C CNN
 F 1 "XBEE_MODULE" H 3750 3250 60  0000 C CNN
-F 2 "" H 4150 2550 60  0001 C CNN
+F 2 "Xbee:XBee_Plug_without_Jtag" H 4150 2550 60  0001 C CNN
 F 3 "" H 4150 2550 60  0001 C CNN
 	1    4150 2550
@@
 NoConn ~ 7150 3200
 NoConn ~ 4950 2600
+$Comp
+L +3V3 #PWR02
+U 1 1 589C012F
+P 3100 2000
+F 0 "#PWR02" H 3100 2225 30  0001 C CNN
+F 1 "+3V3" V 3025 2000 30  0001 C CNN
+F 2 "" H 3100 2000 60  0000 C CNN
+F 3 "" H 3100 2000 60  0000 C CNN
+	1    3100 2000
+	1    0    0    -1
+$EndComp
+$Comp
+L +3V3 #PWR03
+U 1 1 589C0162
+P 5750 3750
+F 0 "#PWR03" H 5750 3975 30  0001 C CNN
+F 1 "+3V3" V 5675 3750 30  0001 C CNN
+F 2 "" H 5750 3750 60  0000 C CNN
+F 3 "" H 5750 3750 60  0000 C CNN
+	1    5750 3750
+	1    0    0    -1
+$EndComp
+$Comp
+L +3V3 #PWR04
+U 1 1 589C03CA
+P 6500 3750
+F 0 "#PWR04" H 6500 3975 30  0001 C CNN
+F 1 "+3V3" V 6425 3750 30  0001 C CNN
+F 2 "" H 6500 3750 60  0000 C CNN
+F 3 "" H 6500 3750 60  0000 C CNN
+	1    6500 3750
+	1    0    0    -1
+$EndComp
+$Comp
+L +3V3 #PWR05
+U 1 1 589C056C
+P 5050 3750
+F 0 "#PWR05" H 5050 3975 30  0001 C CNN
+F 1 "+3V3" V 4975 3750 30  0001 C CNN
+F 2 "" H 5050 3750 60  0000 C CNN
+F 3 "" H 5050 3750 60  0000 C CNN
+	1    5050 3750
+	1    0    0    -1
+$EndComp
+$Comp
+L +3V3 #PWR06
+U 1 1 589C0632
+P 4700 3750
+F 0 "#PWR06" H 4700 3975 30  0001 C CNN
+F 1 "+3V3" V 4625 3750 30  0001 C CNN
+F 2 "" H 4700 3750 60  0000 C CNN
+F 3 "" H 4700 3750 60  0000 C CNN
+	1    4700 3750
+	1    0    0    -1
+$EndComp
+$Comp
+L GNDREF #PWR07
+U 1 1 589C06E2
+P 5350 4500
+F 0 "#PWR07" H 5350 4550 30  0001 C CNN
+F 1 "GNDREF" H 5350 4350 30  0001 C CNN
+F 2 "" H 5350 4500 60  0000 C CNN
+F 3 "" H 5350 4500 60  0000 C CNN
+	1    5350 4500
+	1    0    0    -1
+$EndComp
+$Comp
+L GNDREF #PWR08
+U 1 1 589C0719
+P 4700 4400
+F 0 "#PWR08" H 4700 4450 30  0001 C CNN
+F 1 "GNDREF" H 4700 4250 30  0001 C CNN
+F 2 "" H 4700 4400 60  0000 C CNN
+F 3 "" H 4700 4400 60  0000 C CNN
+	1    4700 4400
+	1    0    0    -1
+$EndComp
+$Comp
+L GNDREF #PWR09
+U 1 1 589C0898
+P 5750 4500
+F 0 "#PWR09" H 5750 4550 30  0001 C CNN
+F 1 "GNDREF" H 5750 4350 30  0001 C CNN
+F 2 "" H 5750 4500 60  0000 C CNN
+F 3 "" H 5750 4500 60  0000 C CNN
+	1    5750 4500
+	1    0    0    -1
+$EndComp
+$Comp
+L GNDREF #PWR010
+U 1 1 589C08C4
+P 6150 4500
+F 0 "#PWR010" H 6150 4550 30  0001 C CNN
+F 1 "GNDREF" H 6150 4350 30  0001 C CNN
+F 2 "" H 6150 4500 60  0000 C CNN
+F 3 "" H 6150 4500 60  0000 C CNN
+	1    6150 4500
+	1    0    0    -1
+$EndComp
+$Comp
+L GNDREF #PWR011
+U 1 1 589C0A71
+P 7600 4650
+F 0 "#PWR011" H 7600 4700 30  0001 C CNN
+F 1 "GNDREF" H 7600 4500 30  0001 C CNN
+F 2 "" H 7600 4650 60  0000 C CNN
+F 3 "" H 7600 4650 60  0000 C CNN
+	1    7600 4650
+	1    0    0    -1
+$EndComp
+$Comp
+L +3V3 #PWR012
+U 1 1 589C0BA4
+P 8050 3750
+F 0 "#PWR012" H 8050 3975 30  0001 C CNN
+F 1 "+3V3" V 7975 3750 30  0001 C CNN
+F 2 "" H 8050 3750 60  0000 C CNN
+F 3 "" H 8050 3750 60  0000 C CNN
+	1    8050 3750
+	1    0    0    -1
+$EndComp
+$Comp
+L R R6
+U 1 1 589C0DAA
+P 8050 4025
+F 0 "R6" V 8130 4025 50  0000 C CNN
+F 1 "1K" V 8050 4025 50  0000 C CNN
+F 2 "Resistors_SMD:R_0805_HandSoldering" V 7980 4025 50  0001 C CNN
+F 3 "" H 8050 4025 50  0000 C CNN
+	1    8050 4025
+	1    0    0    -1
+$EndComp
+$Comp
+L LED D1
+U 1 1 589C0DE1
+P 8050 4425
+F 0 "D1" H 8050 4525 50  0000 C CNN
+F 1 "POWER_LED" H 8050 4325 50  0000 C CNN
+F 2 "LEDs:LED_0805" H 8050 4425 50  0001 C CNN
+F 3 "" H 8050 4425 50  0000 C CNN
+	1    8050 4425
+	0    -1   -1   0
+$EndComp
+$Comp
+L GNDREF #PWR013
+U 1 1 589C0F69
+P 8050 4675
+F 0 "#PWR013" H 8050 4725 30  0001 C CNN
+F 1 "GNDREF" H 8050 4525 30  0001 C CNN
+F 2 "" H 8050 4675 60  0000 C CNN
+F 3 "" H 8050 4675 60  0000 C CNN
+	1    8050 4675
+	1    0    0    -1
+$EndComp
+Wire Wire Line
+	8050 3750 8050 3875
+Wire Wire Line
+	8050 4175 8050 4225
+Wire Wire Line
+	8050 4625 8050 4675
+Wire Wire Line
+	4700 4150 4700 4400
+$Comp
+L +3V3 #PWR014
+U 1 1 589C24FB
+P 5800 2700
+F 0 "#PWR014" H 5800 2925 30  0001 C CNN
+F 1 "+3V3" V 5725 2700 30  0001 C CNN
+F 2 "" H 5800 2700 60  0000 C CNN
+F 3 "" H 5800 2700 60  0000 C CNN
+	1    5800 2700
+	1    0    0    -1
+$EndComp
+$Comp
+L GNDREF #PWR015
+U 1 1 589C2947
+P 8250 2700
+F 0 "#PWR015" H 8250 2750 30  0001 C CNN
+F 1 "GNDREF" H 8250 2550 30  0001 C CNN
+F 2 "" H 8250 2700 60  0000 C CNN
+F 3 "" H 8250 2700 60  0000 C CNN
+	1    8250 2700
+	1    0    0    -1
+$EndComp
 $EndSCHEMATC
